File: Cad designs/PCBs/Main/Main.kicad_pcb (KiCad board)
At the start: 2 copper layers, 68.6 x 53.3 mm, 0 parts

Commit message: 12/08/26
Parts:
- added C1: C, Capacitor_THT:C_Disc_D5.0mm_W2.5mm_P2.50mm, F.Cu at (150.8, 89.5)
- added C2: C, Capacitor_THT:C_Disc_D5.0mm_W2.5mm_P2.50mm, F.Cu at (152.7, 69.2)
- added C3: C, Capacitor_THT:C_Disc_D5.0mm_W2.5mm_P2.50mm, F.Cu at (138.7, 56.2)
- added C4: C, Capacitor_THT:C_Disc_D5.0mm_W2.5mm_P2.50mm, F.Cu at (131.7, 56.2)
- added C5: C, Capacitor_THT:C_Disc_D5.0mm_W2.5mm_P2.50mm, F.Cu at (159.7, 56.2)
- added C6: C, Capacitor_THT:C_Disc_D5.0mm_W2.5mm_P2.50mm, F.Cu at (145.7, 69.2)
- added C7: C, Capacitor_THT:C_Disc_D5.0mm_W2.5mm_P2.50mm, F.Cu at (145.7, 56.2)
- added C8: C, Capacitor_THT:C_Disc_D5.0mm_W2.5mm_P2.50mm, F.Cu at (152.7, 56.2)
- added C9: C, Capacitor_THT:C_Disc_D5.0mm_W2.5mm_P2.50mm, F.Cu at (138.7, 69.2)
- added D1: 1N5819, Diode_THT:D_DO-201AD_P15.24mm_Horizontal, F.Cu at (146.2, 80.0)
- added D2: 1N5819, Diode_THT:D_DO-201AD_P15.24mm_Horizontal, F.Cu at (105.8, 85.3)
- added D3: 1N5819, Diode_THT:D_DO-201AD_P15.24mm_Horizontal, F.Cu at (121.1, 91.3)
- added F1: Polyfuse, Fuse:Fuse_Bourns_MF-RHT050, F.Cu at (126.1, 85.3)
- added F2: Polyfuse, Fuse:Fuse_Bourns_MF-RHT050, F.Cu at (145.7, 84.9)
- added J1: Power, Connector_PinSocket_2.54mm:PinSocket_1x08_P2.54mm_Vertical, F.Cu at (127.9, 97.5)
- added J10: Conn_01x01, Connector_Wire:SolderWire-0.127sqmm_1x01_D0.48mm_OD1mm, F.Cu at (105.5, 48.5)
- added J11: Conn_01x01, Connector_Wire:SolderWire-0.127sqmm_1x01_D0.48mm_OD1mm, F.Cu at (149.2, 53.7)
- added J12: Conn_01x01, Connector_Wire:SolderWire-0.127sqmm_1x01_D0.48mm_OD1mm, F.Cu at (142.2, 65.2)
- added J13: Conn_01x01, Connector_Wire:SolderWire-0.127sqmm_1x01_D0.48mm_OD1mm, F.Cu at (156.2, 65.2)
- added J14: Conn_01x01, Connector_Wire:SolderWire-0.127sqmm_1x01_D0.48mm_OD1mm, F.Cu at (116.5, 71.1)
- added J15: Conn_01x01, Connector_Wire:SolderWire-0.127sqmm_1x01_D0.48mm_OD1mm, F.Cu at (120.2, 71.1)
- added J16: Conn_01x01, Connector_Wire:SolderWire-0.127sqmm_1x01_D0.48mm_OD1mm, F.Cu at (124.0, 71.1)
- added J17: Conn_01x01, Connector_Wire:SolderWire-0.127sqmm_1x01_D0.48mm_OD1mm, F.Cu at (135.2, 53.7)
- added J18: Conn_01x01, Connector_Wire:SolderWire-0.127sqmm_1x01_D0.48mm_OD1mm, F.Cu at (142.2, 53.7)
- added J19: Conn_01x01, Connector_Wire:SolderWire-0.127sqmm_1x01_D0.48mm_OD1mm, F.Cu at (149.2, 65.2)
- added J2: Digital/PWM, Connector_PinSocket_2.54mm:PinSocket_1x10_P2.54mm_Vertical, F.Cu at (118.8, 49.2)
- added J20: Conn_01x01, Connector_Wire:SolderWire-0.127sqmm_1x01_D0.48mm_OD1mm, F.Cu at (109.0, 71.1)
- added J21: Conn_01x01, Connector_Wire:SolderWire-0.127sqmm_1x01_D0.48mm_OD1mm, F.Cu at (112.7, 71.1)
- added J22: Conn_01x01, Connector_Wire:SolderWire-0.127sqmm_1x01_D0.48mm_OD1mm, F.Cu at (149.2, 61.2)
- added J23: Conn_01x01, Connector_Wire:SolderWire-0.127sqmm_1x01_D0.48mm_OD1mm, F.Cu at (149.2, 72.7)
- added J24: Conn_01x01, Connector_Wire:SolderWire-0.127sqmm_1x01_D0.48mm_OD1mm, F.Cu at (124.0, 67.3)
- added J25: Conn_01x01, Connector_Wire:SolderWire-0.127sqmm_1x01_D0.48mm_OD1mm, F.Cu at (120.2, 67.3)
- added J26: Conn_01x01, Connector_Wire:SolderWire-0.127sqmm_1x01_D0.48mm_OD1mm, F.Cu at (109.0, 67.3)
- added J27: Conn_01x01, Connector_Wire:SolderWire-0.127sqmm_1x01_D0.48mm_OD1mm, F.Cu at (135.2, 61.2)
- added J28: Conn_01x01, Connector_Wire:SolderWire-0.127sqmm_1x01_D0.48mm_OD1mm, F.Cu at (163.2, 61.2)
- added J29: Conn_01x01, Connector_Wire:SolderWire-0.127sqmm_1x01_D0.48mm_OD1mm, F.Cu at (142.2, 72.7)
- added J3: Analog, Connector_PinSocket_2.54mm:PinSocket_1x06_P2.54mm_Vertical, F.Cu at (150.8, 97.5)
- added J30: Conn_01x01, Connector_Wire:SolderWire-0.127sqmm_1x01_D0.48mm_OD1mm, F.Cu at (116.5, 67.3)
- added J31: Conn_01x01, Connector_Wire:SolderWire-0.127sqmm_1x01_D0.48mm_OD1mm, F.Cu at (101.8, 48.5)
- added J32: Conn_01x01, Connector_Wire:SolderWire-0.127sqmm_1x01_D0.48mm_OD1mm, F.Cu at (127.7, 67.3)
- added J33: Conn_01x01, Connector_Wire:SolderWire-0.127sqmm_1x01_D0.48mm_OD1mm, F.Cu at (101.8, 52.2)
- added J34: Conn_01x01, Connector_Wire:SolderWire-0.127sqmm_1x01_D0.48mm_OD1mm, F.Cu at (142.2, 61.2)
- added J35: Conn_01x01, Connector_Wire:SolderWire-0.127sqmm_1x01_D0.48mm_OD1mm, F.Cu at (156.2, 61.2)
- added J36: Conn_01x01, Connector_Wire:SolderWire-0.127sqmm_1x01_D0.48mm_OD1mm, F.Cu at (156.2, 72.7)
- added J37: Conn_01x01, Connector_Wire:SolderWire-0.127sqmm_1x01_D0.48mm_OD1mm, F.Cu at (105.2, 67.3)
- added J38: Conn_01x01, Connector_Wire:SolderWire-0.127sqmm_1x01_D0.48mm_OD1mm, F.Cu at (112.7, 67.3)
- added J39: Conn_01x01, Connector_Wire:SolderWire-0.127sqmm_1x01_D0.48mm_OD1mm, F.Cu at (135.2, 57.5)
- added J4: Digital/PWM, Connector_PinSocket_2.54mm:PinSocket_1x08_P2.54mm_Vertical, F.Cu at (145.7, 49.2)
- added J40: Conn_01x01, Connector_Wire:SolderWire-0.127sqmm_1x01_D0.48mm_OD1mm, F.Cu at (142.2, 57.5)
- added J41: Conn_01x01, Connector_Wire:SolderWire-0.127sqmm_1x01_D0.48mm_OD1mm, F.Cu at (149.2, 57.5)
- added J42: Conn_01x01, Connector_Wire:SolderWire-0.127sqmm_1x01_D0.48mm_OD1mm, F.Cu at (156.2, 57.5)
- added J43: Conn_01x01, Connector_Wire:SolderWire-0.127sqmm_1x01_D0.48mm_OD1mm, F.Cu at (163.2, 57.5)
- added J44: Conn_01x01, Connector_Wire:SolderWire-0.127sqmm_1x01_D0.48mm_OD1mm, F.Cu at (142.2, 69.0)
- added J45: Conn_01x01, Connector_Wire:SolderWire-0.127sqmm_1x01_D0.48mm_OD1mm, F.Cu at (149.2, 69.0)
- added J46: Conn_01x01, Connector_Wire:SolderWire-0.127sqmm_1x01_D0.48mm_OD1mm, F.Cu at (156.2, 69.0)
- added J47: Conn_01x01, Connector_Wire:SolderWire-0.127sqmm_1x01_D0.48mm_OD1mm, F.Cu at (101.8, 87.5)
- added J48: Conn_01x01, Connector_Wire:SolderWire-0.127sqmm_1x01_D0.48mm_OD1mm, F.Cu at (165.9, 80.8)
- added J49: Conn_01x01, Connector_Wire:SolderWire-0.127sqmm_1x01_D0.48mm_OD1mm, F.Cu at (165.9, 84.5)
- added J5: Conn_01x01, Connector_Wire:SolderWire-0.127sqmm_1x01_D0.48mm_OD1mm, F.Cu at (156.2, 53.7)
- added J50: Conn_01x01, Connector_Wire:SolderWire-0.127sqmm_1x01_D0.48mm_OD1mm, F.Cu at (101.8, 91.3)
- added J6: Conn_01x01, Connector_Wire:SolderWire-0.127sqmm_1x01_D0.48mm_OD1mm, F.Cu at (163.2, 53.7)
- added J7: Conn_01x01, Connector_Wire:SolderWire-0.127sqmm_1x01_D0.48mm_OD1mm, F.Cu at (105.2, 71.1)
- added J8: Conn_01x01, Connector_Wire:SolderWire-0.127sqmm_1x01_D0.48mm_OD1mm, F.Cu at (127.7, 71.1)
- added J9: Conn_01x01, Connector_Wire:SolderWire-0.127sqmm_1x01_D0.48mm_OD1mm, F.Cu at (105.5, 52.2)
- added R1: R, Resistor_THT:R_Axial_DIN0207_L6.3mm_D2.5mm_P7.62mm_Horizontal, F.Cu at (124.2, 64.3)
- added R2: R, Resistor_THT:R_Axial_DIN0207_L6.3mm_D2.5mm_P7.62mm_Horizontal, F.Cu at (121.2, 56.7)
- added R3: R, Resistor_THT:R_Axial_DIN0207_L6.3mm_D2.5mm_P7.62mm_Horizontal, F.Cu at (118.2, 56.7)
- added R4: R, Resistor_THT:R_Axial_DIN0207_L6.3mm_D2.5mm_P7.62mm_Horizontal, F.Cu at (114.2, 56.7)
- added R5: R, Resistor_THT:R_Axial_DIN0207_L6.3mm_D2.5mm_P7.62mm_Horizontal, F.Cu at (111.2, 56.7)
- added R6: R, Resistor_THT:R_Axial_DIN0207_L6.3mm_D2.5mm_P7.62mm_Horizontal, F.Cu at (108.2, 56.7)
- added R7: R, Resistor_THT:R_Axial_DIN0207_L6.3mm_D2.5mm_P7.62mm_Horizontal, F.Cu at (105.2, 64.3)
- added R8: R, Resistor_THT:R_Axial_DIN0207_L6.3mm_D2.5mm_P7.62mm_Horizontal, F.Cu at (153.8, 85.5)
- added R9: R, Resistor_THT:R_Axial_DIN0207_L6.3mm_D2.5mm_P7.62mm_Horizontal, F.Cu at (153.8, 89.5)
Routing:
- net 0: track 649.7 -> 0.00 mm
- net /*10: track 0.00 -> 129.3 mm
- net (no net): track 0.00 -> 127.8 mm
- net /A1: track 0.00 -> 38.5 mm
- net /A2: track 0.00 -> 34.9 mm
- net /A3: track 0.00 -> 33.0 mm
- net Net-(J4-Pin_1): track 0.00 -> 25.4 mm
- net /8: track 0.00 -> 23.6 mm
- net /*6: track 0.00 -> 22.9 mm
- net /SDA/A4: track 0.00 -> 21.6 mm
- net /A0: track 0.00 -> 20.4 mm
- net VCC: track 0.00 -> 19.1 mm
- net /*5: track 0.00 -> 18.3 mm
- net /2: track 0.00 -> 17.6 mm
- net /SCL/A5: track 0.00 -> 15.0 mm
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- added copper zone on F.Cu, net +5V
- added copper zone on B.Cu, net GND
