File: Cad designs/PCBs/PPTC/PPTC PCB/PPTC PCB.kicad_sch (KiCad schematic)
At the start: 4 parts, among them J1 Power, J2 Digital/PWM, J3 Analog, J4 Digital/PWM

Commit message: 1
Parts:
- removed J1: Power, Connector_PinSocket_2.54mm:PinSocket_1x08_P2.54mm_Vertical, symbol Connector_Generic:Conn_01x08
- removed J2: Digital/PWM, Connector_PinSocket_2.54mm:PinSocket_1x10_P2.54mm_Vertical, symbol Connector_Generic:Conn_01x10
- removed J3: Analog, Connector_PinSocket_2.54mm:PinSocket_1x06_P2.54mm_Vertical, symbol Connector_Generic:Conn_01x06
- removed J4: Digital/PWM, Connector_PinSocket_2.54mm:PinSocket_1x08_P2.54mm_Vertical, symbol Connector_Generic:Conn_01x08
- added F1: Polyfuse, Fuse:Fuse_Bourns_MF-RHT050, symbol Device:Polyfuse
- added J1, J2, J3, J4: Conn_01x01, Connector_PinHeader_1.00mm:PinHeader_1x01_P1.00mm_Vertical, symbol Connector_Generic:Conn_01x01
Connections:
- new net: F1.1, J3.1 (Pin_1)
- new net: J2.1 (Pin_1), J4.1 (Pin_1)
- new net: F1.2, J1.1 (Pin_1)
- no-connect marks 1 -> 0
